File: f_buzzer.sch (KiCad schematic (older format))
At the start: 10 parts, among them U1 SN74LS123DRG4

Commit message: Updated the schematics and pcb design
Parts:
- RV1: footprint f_buzzer:Potentiometer_Bourns_3345P_Horizontal -> f_buzzer:VG039NCHXTB203; LCSC (none) -> C128550
Changed lines of the file:
@@
 F 0 "RV1" V 6943 4200 50  0000 C CNN
 F 1 "20K" V 7034 4200 50  0000 C CNN
-F 2 "f_buzzer:Potentiometer_Bourns_3345P_Horizontal" H 7150 4200 50  0001 C CNN
-F 3 "~" H 7150 4200 50  0001 C CNN
+F 2 "f_buzzer:VG039NCHXTB203" H 7150 4200 50  0001 C CNN
+F 3 "https://datasheet.lcsc.com/szlcsc/1810170727_HDK-Hokuriku-Elec-Industry-VG039NCHXTB203_C128550.pdf" H 7150 4200 50  0001 C CNN
+F 4 "C128550" V 7150 4200 50  0001 C CNN "LCSC"
 	1    7150 4200
 	0    1    1    0
